Commit message: added functionality for gazebo launch and is working now

File: src/robot_description/urdf/robot.urdf.xacro (robot description, xacro)
@@ -1,4 +1,5 @@
 <?xml version="1.0"?>
 <robot name="robot" xmlns:xacro="http://ros.org/wiki/xacro">
+    <xacro:include filename="$(find robot_description)/urdf/robot_gazebo.xacro" />
     <material name="blue">
         <color rgba="0 0 1 1"/>
@@ -30,4 +31,5 @@
             </geometry>
             <origin xyz="0 0 0.0015" rpy="0 0 1.57"/>
+            <material name="black"/>
         </visual>
         <collision>
@@ -51,4 +53,5 @@
             </geometry>
             <origin xyz="0 0 0" rpy="0 0 0"/>
+            <material name="dark_grey"/>
         </visual>
         <collision>
@@ -118,4 +121,5 @@
             </geometry>
             <origin xyz="0 0 0" rpy="0 0 1.57"/>
+            <material name="silver"/>
         </visual>
         <collision>
@@ -139,4 +143,5 @@
             </geometry>
             <origin xyz="0 0 0" rpy="0 0 1.57"/>
+            <material name="silver"/>
         </visual>
         <collision>
