Commit message: added robot_cpp_examples and robot_py_examples and also added robot_controller pkgs for support for controllers but it is not working

File: src/robot_description/urdf/robot_gazebo.xacro (robot description, xacro)
@@ -1,5 +1,5 @@
 <?xml version="1.0"?>
 <robot name="robot" xmlns:xacro="http://ros.org/wiki/xacro">
-  <!-- Wheels -->
+    <!-- Wheels -->
   <gazebo reference="wheel_left_link">
     <mu1>1000000000000000.0</mu1>
@@ -40,10 +40,10 @@
     <xacro:if value="$(arg is_ignition)"><!--if user has ros2 humble and ingition gazebo-->
       <plugin filename="ign_ros2_control-system" name="ign_ros2_control::IgnitionROS2ControlPlugin"> <!-- loading ignition gazebo control system bcuz user has ros2 humble-->
-        <parameters></parameters>
+        <parameters>$(find robot_controller)/config/robot_controllers.yaml</parameters> <!-- loading yaml file from robot_controller pkg into ros2_control system-->
       </plugin>
     </xacro:if>
     <xacro:unless value="$(arg is_ignition)"> <!-- if user has ros2 jazzy and gazebo-->
-      <plugin filename="gz_ros2_control-system" name="gz_ros2_control::GazeboROS2ControlPlugin"> <!-- loading gazebo control system bcuz user has ros2 jazzy-->
-        <parameters></parameters>
+      <plugin filename="gz_ros2_control-system" name="gz_ros2_control::GazeboSimROS2ControlPlugin"> <!-- loading gazebo control system bcuz user has ros2 jazzy-->
+        <parameters>$(find robot_controller)/config/robot_controllers.yaml</parameters> <!-- loading yaml file from robot_controller pkg into ros2_control system-->
       </plugin>
     </xacro:unless>

File: src/robot_description/urdf/robot_ros2_control.xacro (robot description, xacro)
@@ -1,34 +1,32 @@
 <?xml version="1.0"?>
-<robot name="robot" xmlns:xacro="http://ros.org/wiki/xacro">
+<robot xmlns:xacro="http://www.ros.org/wiki/xacro" name="robot">
     <ros2_control name="RobotSystem" type="system">
-        <xacro:if value="$(arg is_ignition)"> <!--if user has ros2 humble and ingition gazebo-->
+        <xacro:if value="$(arg is_ignition)">
             <hardware>
                 <plugin>ign_ros2_control/IgnitionSystem</plugin>
             </hardware>
         </xacro:if>
-        <xacro:unless value="$(arg is_ignition)"> <!-- if user has ros2 jazzy and gazebo-->
-             <hardware>
+        <xacro:unless value="$(arg is_ignition)">
+            <hardware>
                 <plugin>gz_ros2_control/GazeboSimSystem</plugin>
             </hardware>
         </xacro:unless>
-        <joint name="wheel_right_joint"> <!-- defining joinst which the ros2_control pkg will control-->
+        <joint name="wheel_right_joint">
+            <command_interface name="velocity">
+              <param name="min">-1</param>
+              <param name="max">1</param>
+            </command_interface>
+            <state_interface name="position" />
+            <state_interface name="velocity" />
+        </joint>
+        <joint name="wheel_left_joint">
             <!-- command interface means the inetrface through which we will send commands for wheels to rotate-->
             <!-- state interface means the interface through which we will read the state of the motors-->
             <command_interface name="velocity"> <!-- defining the interfaces we want for wheel-->
-                <param name="min">-1</param> <!-- max limit for motor.. value is in rad/sec-->
-                <param name="max">1</param> <!-- min limit for motor.. value is in rad/sec-->
+              <param name="min">-1</param> <!-- min limit for motor.. value is in rad/sec-->
+              <param name="max">1</param> <!-- max limit for motor.. value is in rad/sec-->
             </command_interface>
-            <state_interface name="position"/>
-            <state_interface name="velocity"/>
-        </joint>
-        <joint name="wheel_left_joint"> <!-- defining joinst which the ros2_control pkg will control-->
-            <!-- command interface means the inetrface through which we will send commands for wheels to rotate-->
-            <!-- state interface means the interface through which we will read the state of the motors-->
-            <command_interface name="velocity"> <!-- defining the interfaces we want for wheel-->
-                <param name="min">-1</param> <!-- max limit for motor.. value is in rad/sec-->
-                <param name="max">1</param> <!-- min limit for motor.. value is in rad/sec-->
-            </command_interface>
-            <state_interface name="position"/>
-            <state_interface name="velocity"/>
+            <state_interface name="position" />
+            <state_interface name="velocity" />
         </joint>
     </ros2_control>
