Commit message: renamed robot_description pkg to bumperbot_description and changed plugins... error of failed activation not solved

File: src/bumperbot_description/urdf/robot.urdf.xacro (robot description, xacro)
@@ -4,7 +4,7 @@
     <xacro:arg name="is_ignition" default="true"/>
     <!-- including gazebo parameters from file-->
-    <xacro:include filename="$(find robot_description)/urdf/robot_gazebo.xacro" />
+    <xacro:include filename="$(find bumperbot_description)/urdf/robot_gazebo.xacro" />
     <!-- including ros2_control parametersfrom file-->
-    <xacro:include filename="$(find robot_description)/urdf/robot_ros2_control.xacro" />
+    <xacro:include filename="$(find bumperbot_description)/urdf/robot_ros2_control.xacro" />
     <material name="blue">
         <color rgba="0 0 1 1"/>
@@ -33,5 +33,5 @@
         <visual>
             <geometry>
-                <mesh filename="package://robot_description/meshes/base_link.stl" scale="0.001 0.001 0.001"/>
+                <mesh filename="package://bumperbot_description/meshes/base_link.stl" scale="0.001 0.001 0.001"/>
             </geometry>
             <origin xyz="0 0 0.0015" rpy="0 0 1.57"/>
@@ -40,5 +40,5 @@
         <collision>
             <geometry>
-                <mesh filename="package://robot_description/meshes/base_link.stl" scale="0.001 0.001 0.001"/>
+                <mesh filename="package://bumperbot_description/meshes/base_link.stl" scale="0.001 0.001 0.001"/>
             </geometry>
             <origin xyz="0 0 0.0015" rpy="0 0 1.57"/>
@@ -55,5 +55,5 @@
         <visual>
             <geometry>
-                <mesh filename="package://robot_description/meshes/new_laser_link.stl"/>
+                <mesh filename="package://bumperbot_description/meshes/new_laser_link.stl"/>
             </geometry>
             <origin xyz="0 0 0" rpy="0 0 0"/>
@@ -62,5 +62,5 @@
         <collision>
             <geometry>
-                <mesh filename="package://robot_description/meshes/new_laser_link.stl"/>
+                <mesh filename="package://bumperbot_description/meshes/new_laser_link.stl"/>
             </geometry>
             <origin xyz="0 0 0" rpy="0 0 0"/>
@@ -77,5 +77,5 @@
         <visual>
             <geometry>
-                <mesh filename="package://robot_description/meshes/wheel_right_link.stl" scale="0.001 0.001 0.001"/>
+                <mesh filename="package://bumperbot_description/meshes/wheel_right_link.stl" scale="0.001 0.001 0.001"/>
             </geometry>
             <origin xyz="0 0 0" rpy="-1.57 0 0"/>
@@ -84,5 +84,5 @@
         <collision>
             <geometry>
-                <mesh filename="package://robot_description/meshes/wheel_right_link.stl" scale="0.001 0.001 0.001"/>
+                <mesh filename="package://bumperbot_description/meshes/wheel_right_link.stl" scale="0.001 0.001 0.001"/>
             </geometry>
             <origin xyz="0 0 0" rpy="-1.57 0 0"/>
@@ -100,5 +100,5 @@
         <visual>
             <geometry>
-                <mesh filename="package://robot_description/meshes/wheel_left_link.stl" scale="0.001 0.001 0.001"/>
+                <mesh filename="package://bumperbot_description/meshes/wheel_left_link.stl" scale="0.001 0.001 0.001"/>
             </geometry>
             <origin xyz="0 0 0" rpy="1.57 0 0"/>
@@ -107,5 +107,5 @@
         <collision>
             <geometry>
-                <mesh filename="package://robot_description/meshes/wheel_left_link.stl" scale="0.001 0.001 0.001"/>
+                <mesh filename="package://bumperbot_description/meshes/wheel_left_link.stl" scale="0.001 0.001 0.001"/>
             </geometry>
             <origin xyz="0 0 0" rpy="1.57 0 0"/>
@@ -123,5 +123,5 @@
         <visual>
             <geometry>
-                <mesh filename="package://robot_description/meshes/caster_rear_link.stl" scale="0.001 0.001  0.001"/>
+                <mesh filename="package://bumperbot_description/meshes/caster_rear_link.stl" scale="0.001 0.001  0.001"/>
             </geometry>
             <origin xyz="0 0 0" rpy="0 0 1.57"/>
@@ -130,5 +130,5 @@
         <collision>
             <geometry>
-                <mesh filename="package://robot_description/meshes/caster_rear_link.stl" scale="0.001 0.001  0.001"/>
+                <mesh filename="package://bumperbot_description/meshes/caster_rear_link.stl" scale="0.001 0.001  0.001"/>
             </geometry>
             <origin xyz="0 0 0" rpy="0 0 1.57"/>
@@ -145,5 +145,5 @@
         <visual>
             <geometry>
-                <mesh filename="package://robot_description/meshes/caster_front_link.stl" scale="0.001 0.001  0.001"/>
+                <mesh filename="package://bumperbot_description/meshes/caster_front_link.stl" scale="0.001 0.001  0.001"/>
             </geometry>
             <origin xyz="0 0 0" rpy="0 0 1.57"/>
@@ -152,5 +152,5 @@
         <collision>
             <geometry>
-                <mesh filename="package://robot_description/meshes/caster_front_link.stl" scale="0.001 0.001  0.001"/>
+                <mesh filename="package://bumperbot_description/meshes/caster_front_link.stl" scale="0.001 0.001  0.001"/>
             </geometry>
             <origin xyz="0 0 0" rpy="0 0 1.57"/>

File: src/bumperbot_description/urdf/robot_gazebo.xacro (robot description, xacro)
@@ -38,14 +38,7 @@
   </gazebo>
   <gazebo><!-- checking if user has ignition gazebo or not-->
-    <xacro:if value="$(arg is_ignition)"><!--if user has ros2 humble and ingition gazebo-->
-      <plugin filename="ign_ros2_control-system" name="ign_ros2_control::IgnitionROS2ControlPlugin"> <!-- loading ignition gazebo control system bcuz user has ros2 humble-->
-        <parameters>$(find robot_controller)/config/robot_controllers.yaml</parameters> <!-- loading yaml file from robot_controller pkg into ros2_control system-->
-      </plugin>
-    </xacro:if>
-    <xacro:unless value="$(arg is_ignition)"> <!-- if user has ros2 jazzy and gazebo-->
-      <plugin filename="gz_ros2_control-system" name="gz_ros2_control::GazeboSimROS2ControlPlugin"> <!-- loading gazebo control system bcuz user has ros2 jazzy-->
-        <parameters>$(find robot_controller)/config/robot_controllers.yaml</parameters> <!-- loading yaml file from robot_controller pkg into ros2_control system-->
-      </plugin>
-    </xacro:unless>
+    <plugin filename="ign_ros2_control-system" name="ign_ros2_control::IgnitionROS2ControlPlugin">
+    <parameters>$(find robot_controller)/config/robot_controllers.yaml</parameters>
+    </plugin>
   </gazebo>
 </robot>

File: src/bumperbot_description/urdf/robot_ros2_control.xacro (robot description, xacro)
@@ -4,15 +4,7 @@
         <!-- ros2_control Gazebo -->
         <!-- ROS 2 Humble -->
-        <xacro:if value="$(arg is_ignition)">
-            <hardware>
-                <plugin>ign_ros2_control/IgnitionSystem</plugin>
-            </hardware>
-        </xacro:if>
-        <!-- ROS 2 Iron or above -->
-        <xacro:unless value="$(arg is_ignition)">
-            <hardware>
-                <plugin>gz_ros2_control/GazeboSimSystem</plugin>
-            </hardware>
-        </xacro:unless>
+        <hardware>
+            <plugin>ign_ros2_control/IgnitionSystem</plugin>
+        </hardware>
         <!-- ros2_control Common Interfaces -->
         <joint name="wheel_right_joint">
