Commit message: found a new urdf issue... solved it and added support for joystick but robot not moving in gazebo

File: src/bumperbot_description/urdf/bumperbot.urdf.xacro (robot description, xacro)
@@ -115,5 +115,5 @@
   </link>
   <joint name="caster_front_joint" type="fixed">
-    <origin xyz="0.0762 0 -0.0345011" rpy="0 0 0" />
+    <origin xyz="0.0762 0 -0.0380011" rpy="0 0 0" />
     <parent link="base_link" />
     <child link="caster_front_link" />
@@ -142,5 +142,5 @@
   </link>
   <joint name="caster_rear_joint" type="fixed">
-    <origin xyz="0.0762 0 -0.0345011" rpy="0 0 0" />
+    <origin xyz="-0.0762 0 -0.0380011" rpy="0 0 0" />
     <parent link="base_link" />
     <child link="caster_rear_link" />

Commit message: tuned inertia and collision tags

File: src/bumperbot_description/urdf/bumperbot.urdf.xacro (robot description, xacro)
@@ -51,7 +51,7 @@
     </visual>
     <collision>
-      <origin xyz="0 0 0" rpy="-1.57 0 0" />
+      <origin xyz="0 0.008 0" rpy="-1.57 0 0" />
       <geometry>
-        <mesh filename="package://bumperbot_description/meshes/wheel_right_link.stl" scale="0.001 0.001 0.001"/>
+        <cylinder radius="0.0534" length="0.0285"/>
       </geometry>
     </collision>
@@ -80,7 +80,7 @@
     </visual>
     <collision>
-      <origin xyz="0 0.015 0" rpy="1.57 0 0" />
+      <origin xyz="0 -0.009 0" rpy="1.57 0 0" />
       <geometry>
-        <mesh filename="package://bumperbot_description/meshes/wheel_left_link.stl" scale="0.001 0.001 0.001"/>
+        <cylinder radius="0.0534" length="0.0285"/>
       </geometry>
     </collision>
@@ -108,7 +108,7 @@
     </visual>
     <collision>
-      <origin xyz="0 0 0" rpy="0 0 1.57" />
+      <origin xyz="0 0 0.0211305" rpy="0 0 0" />
       <geometry>
-        <mesh filename="package://bumperbot_description/meshes/caster_front_link.stl" scale="0.001 0.001  0.001"/>
+        <sphere radius="0.0211305"/>
       </geometry>
     </collision>
@@ -135,7 +135,7 @@
     </visual>
     <collision>
-      <origin xyz="0 0 0" rpy="0 0 1.57" />
+      <origin xyz="0 0 0.0211305" rpy="0 0 0" />
       <geometry>
-        <mesh filename="package://bumperbot_description/meshes/caster_rear_link.stl" scale="0.001 0.001  0.001"/>
+        <sphere radius="0.0211305"/>
       </geometry>
     </collision>
@@ -163,7 +163,7 @@
         <collision>
             <geometry>
-                <mesh filename="package://bumperbot_description/meshes/new_laser_link.stl"/>
+                <box size="0.071689 0.097337 0.05350"/>
             </geometry>
-            <origin xyz="0 0 0" rpy="0 0 0"/>
+            <origin xyz="0 0 -0.015" rpy="0 0 0"/>
         </collision>
     </link>

Commit message: fine tuned more values and changed inertia values

File: src/bumperbot_description/urdf/bumperbot.urdf.xacro (robot description, xacro)
@@ -10,21 +10,21 @@
   <link name="base_link">
     <inertial>
-      <origin xyz="0.0065 0.002607 0.020274" rpy="0 0 0"/>
-      <mass value="0.947792"/>
-      <inertia ixx="3.036"    ixy="-0.4767"  ixz="-0.511"
-               iyy="1.659"    iyz="-1.036"
-               izz="3.374" />
+      <origin xyz="0.000392694 0.003603923 0.028354103" rpy="0 0 0"/>
+      <mass value="1.1796479"/>
+      <inertia ixx="0.010666756"    ixy="0.000115581"  ixz="0.001086391"
+               iyy="0.011710101"    iyz="-0.000017452"
+               izz="0.00663569" />
     </inertial>
     <visual>
-      <origin xyz="0 0 0.0015" rpy="0 0 1.57" />
-      <material name="black"/>
+      <origin xyz="0 0 0.0015" rpy="0 0 0" />
+      <!-- <material name="black"/> -->
       <geometry>
-        <mesh filename="package://bumperbot_description/meshes/base_link.stl" scale="0.001 0.001 0.001"/>
+        <mesh filename="package://bumperbot_description/meshes/base_link.stl"/>
       </geometry>
     </visual>
     <collision>
-      <origin xyz="0 0 0.0015" rpy="0 0 1.57" />
+      <origin xyz="0 0 0.0015" rpy="0 0 0" />
       <geometry>
-        <mesh filename="package://bumperbot_description/meshes/base_link.stl" scale="0.001 0.001 0.001"/>
+        <mesh filename="package://bumperbot_description/meshes/base_link.stl"/>
       </geometry>
     </collision>
@@ -36,20 +36,20 @@
   </joint>
   <link name="wheel_right_link">
-    <inertial>
-      <origin xyz="6.671e-12 -1.094e-11 0.012102" rpy="0 0 0"/>
-      <mass value="0.09205" />
-      <inertia ixx="9.3607e-05"  ixy="-4.428e-15"  ixz="6.941e-16"
-               iyy="9.3607e-05"  iyz="-1.133e-15"
-               izz="1.802e-04" />
+   <inertial>
+      <origin xyz="0 9.713661142e-10 0.016398450" rpy="0 0 0" />
+      <mass value="0.092049771" />
+      <inertia ixx="0.000093607"  ixy="0"  ixz="0"
+               iyy="0.000093607"  iyz="0"
+               izz="0.000180163" />
     </inertial>
     <visual>
-      <origin xyz="0 0 0" rpy="-1.57 0 0" />
+      <origin xyz="0 0 0" rpy="1.57 0 0" />
       <material name="blue" />
       <geometry>
-        <mesh filename="package://bumperbot_description/meshes/wheel_right_link.stl" scale="0.001 0.001 0.001"/>
+        <mesh filename="package://bumperbot_description/meshes/wheel_right_link.stl"/>
       </geometry>
     </visual>
     <collision>
-      <origin xyz="0 0.008 0" rpy="-1.57 0 0" />
+      <origin xyz="0 -0.017 0" rpy="1.57 0 0" />
       <geometry>
         <cylinder radius="0.0534" length="0.0285"/>
@@ -58,5 +58,5 @@
   </link>
   <joint name="wheel_right_joint" type="continuous">
-    <origin xyz="0 -0.14355 0.015" rpy="0 0 0" />
+    <origin xyz="0 -0.11455 0.015" rpy="0 0 0" />
     <parent link="base_link" />
     <child link="wheel_right_link" />
@@ -66,19 +66,19 @@
     name="wheel_left_link">
     <inertial>
-      <origin xyz="6.671e-12 -1.094e-11 0.012102" rpy="0 0 0" />
-      <mass value="0.09205" />
-      <inertia ixx="9.3607e-05"  ixy="-4.428e-15"  ixz="6.941e-16"
-               iyy="9.3607e-05"  iyz="-1.133e-15"
-               izz="1.802e-04" />
+      <origin xyz="0 9.713661142e-10 0.016398450" rpy="0 0 0" />
+      <mass value="0.092049771" />
+      <inertia ixx="0.000093607"  ixy="0"  ixz="0"
+               iyy="0.000093607"  iyz="0"
+               izz="0.000180163" />
     </inertial>
     <visual>
-      <origin xyz="0 0 0" rpy="1.57 0 0" />
+      <origin xyz="0 0 0" rpy="-1.57 0 0" />
       <material name="blue" />
       <geometry>
-        <mesh filename="package://bumperbot_description/meshes/wheel_left_link.stl" scale="0.001 0.001 0.001"/>
+        <mesh filename="package://bumperbot_description/meshes/wheel_left_link.stl"/>
       </geometry>
     </visual>
     <collision>
-      <origin xyz="0 -0.009 0" rpy="1.57 0 0" />
+      <origin xyz="0 0.017 0" rpy="-1.57 0 0" />
       <geometry>
         <cylinder radius="0.0534" length="0.0285"/>
@@ -87,5 +87,5 @@
   </link>
   <joint name="wheel_left_joint" type="continuous">
-    <origin xyz="0 0.14355 0.015" rpy="0 0 0" />
+    <origin xyz="0 0.11455 0.015" rpy="0 0 0" />
     <parent link="base_link" />
     <child link="wheel_left_link" />
@@ -94,9 +94,9 @@
   <link name="caster_front_link">
     <inertial>
-      <origin xyz="0.000348 -0.003895 0.018625" rpy="0 0 0" />
-      <mass value="0.030003" />
-      <inertia ixx="5.032352e-06"  ixy="7.6e-10"    ixz="-5.91e-10"
-               iyy="5.178243e-06"  iyz="-2.92e-10"
-               izz="5.249228e-06" />
+      <origin xyz="-0.055462489 0.004963490 0.019704843" rpy="0 0 0" />
+      <mass value="0.034768653" />
+      <inertia ixx="0.000006952"  ixy="-8.168396889e-10"    ixz="4.36638148e-10"
+               iyy="0.00000631"  iyz="-8.101927285e-10"
+               izz="0.000006556" />
     </inertial>
     <visual>
@@ -104,9 +104,9 @@
       <material name="silver"/>
       <geometry>
-        <mesh filename="package://bumperbot_description/meshes/caster_front_link.stl" scale="0.001 0.001  0.001"/>
+        <mesh filename="package://bumperbot_description/meshes/caster_front_link.stl"/>
       </geometry>
     </visual>
     <collision>
-      <origin xyz="0 0 0.0211305" rpy="0 0 0" />
+      <origin xyz="0 0 0.0211305" rpy="0 0 1.57" />
       <geometry>
         <sphere radius="0.0211305"/>
@@ -121,9 +121,9 @@
   <link name="caster_rear_link">
     <inertial>
-      <origin xyz="0.000348 -0.003895 0.018625" rpy="0 0 0" />
-      <mass value="0.030003" />
-      <inertia ixx="5.032352e-06"  ixy="7.6e-10"    ixz="-5.91e-10"
-               iyy="5.178243e-06"  iyz="-2.92e-10"
-               izz="5.249228e-06" />
+      <origin xyz="-0.055462489 0.004963490 0.019704843" rpy="0 0 0" />
+      <mass value="0.034768653" />
+      <inertia ixx="0.000006952"  ixy="-8.168396889e-10"    ixz="4.36638148e-10"
+               iyy="0.00000631"  iyz="-8.101927285e-10"
+               izz="0.000006556" />
     </inertial>
     <visual>
@@ -131,9 +131,9 @@
       <material name="silver"/>
       <geometry>
-        <mesh filename="package://bumperbot_description/meshes/caster_rear_link.stl" scale="0.001 0.001  0.001"/>
+        <mesh filename="package://bumperbot_description/meshes/caster_rear_link.stl"/>
       </geometry>
     </visual>
     <collision>
-      <origin xyz="0 0 0.0211305" rpy="0 0 0" />
+      <origin xyz="0 0 0.0211305" rpy="0 0 1.57" />
       <geometry>
         <sphere radius="0.0211305"/>

Commit message: added imu in urdf and in _gazzebo.xacro, added ros2 gz bridge support for imu also, code is working, urdf values are finetuned

File: src/bumperbot_description/urdf/bumperbot.urdf.xacro (robot description, xacro)
@@ -168,9 +168,34 @@
         </collision>
     </link>
-    <joint name="laser_joint" type="fixed">
+  <joint name="laser_joint" type="fixed">
         <origin xyz="0 0 0.131" rpy="0 0 0" /> <!-- z= 0.042(from physical unit) + 0.088(from fusion final assembly without wheels) + 0.001(accounting for plate thickness)-->
         <parent link="base_link" />
         <child link="laser" />
-    </joint>
+  </joint>
+  <link name="imu_link">
+    <inertial>
+      <origin xyz="-0.057000001 -0.076500001 0.048500000" rpy="0.0 0.0 0.0"/>
+      <mass value="0.001307313"/>
+      <inertia ixx="4.630065354e-08" ixy="0.0" ixz="0.0" iyy="2.723567855e-08" iyz="0.0" izz="6.808919639e-08"/>
+    </inertial>
+    <visual>
+      <origin xyz="0 0 0" rpy="0 0 0" />
+      <material name="amber_gold"/>
+      <geometry>
+        <mesh filename="package://bumperbot_description/meshes/imu_link.STL"/>
+      </geometry>
+    </visual>
+    <collision>
+      <origin xyz="0 0 0" rpy="0 0 0" />
+      <geometry>
+        <box size="0.02 0.015 0.005"/>
+      </geometry>
+    </collision>
+  </link>
+  <joint name="imu_joint" type="fixed">
+    <parent link="base_link"/>
+    <child link="imu_link"/>
+    <origin xyz="-0.020000 -0.08000 0.04780000" rpy="0.0 0.0 0.0"/> <!-- x and y values from fusion and z value is from fusion but also adjusted-->
+  </joint>
   <material name="blue">
     <color rgba="0 0 1 1"/>

File: src/bumperbot_description/urdf/bumperbot_gazebo.xacro (robot description, xacro)
@@ -44,4 +44,5 @@
         <parameters>$(find bumperbot_controller)/config/bumperbot_controllers.yaml</parameters>
       </plugin>
+      <plugin filename="ignition-gazebo-imu-system" name="ignition::gazebo::systems::Imu"></plugin>
     </xacro:if>
     <!-- ROS 2 Iron or above -->
@@ -50,5 +51,57 @@
         <parameters>$(find bumperbot_controller)/config/bumperbot_controllers.yaml</parameters>
       </plugin>
+      <plugin filename="gz-sim-imu-system" name="gz::sim::systems::Imu"></plugin>
     </xacro:unless>
   </gazebo>
+    <!-- IMU -->
+  <gazebo reference="imu_link">
+    <sensor name="imu" type="imu">
+        <always_on>true</always_on>
+        <update_rate>100</update_rate>
+        <gz_frame_id>imu_link</gz_frame_id>
+        <topic>imu</topic>
+        <imu>
+          <angular_velocity>
+            <x>
+              <noise type="gaussian">
+                <mean>0.0</mean>
+                <stddev>2e-4</stddev>
+              </noise>
+            </x>
+            <y>
+              <noise type="gaussian">
+                <mean>0.0</mean>
+                <stddev>2e-4</stddev>
+              </noise>
+            </y>
+            <z>
+              <noise type="gaussian">
+                <mean>0.0</mean>
+                <stddev>2e-4</stddev>
+              </noise>
+            </z>
+          </angular_velocity>
+          <linear_acceleration>
+            <x>
+              <noise type="gaussian">
+                <mean>0.0</mean>
+                <stddev>1.7e-2</stddev>
+              </noise>
+            </x>
+            <y>
+              <noise type="gaussian">
+                <mean>0.0</mean>
+                <stddev>1.7e-2</stddev>
+              </noise>
+            </y>
+            <z>
+              <noise type="gaussian">
+                <mean>0.0</mean>
+                <stddev>1.7e-2</stddev>
+              </noise>
+            </z>
+          </linear_acceleration>
+        </imu>
+    </sensor>
+  </gazebo>
 </robot>

Commit message: chnaged base_link,stl to match imu, now working, moving on to solve odom error in section 11 odometry and control

File: src/bumperbot_description/urdf/bumperbot.urdf.xacro (robot description, xacro)
@@ -20,5 +20,5 @@
       <!-- <material name="black"/> -->
       <geometry>
-        <mesh filename="package://bumperbot_description/meshes/base_link.stl"/>
+        <mesh filename="package://bumperbot_description/meshes/base_link.stl" scale="0.001 0.001 0.001"/>
       </geometry>
     </visual>
@@ -26,5 +26,5 @@
       <origin xyz="0 0 0.0015" rpy="0 0 0" />
       <geometry>
-        <mesh filename="package://bumperbot_description/meshes/base_link.stl"/>
+        <mesh filename="package://bumperbot_description/meshes/base_link.stl" scale="0.001 0.001 0.001"/>
       </geometry>
     </collision>

Commit message: fixed orientaion of lidar in urdf

File: src/bumperbot_description/urdf/bumperbot.urdf.xacro (robot description, xacro)
@@ -148,27 +148,27 @@
   </joint>
   <link name="laser">
-        <inertial>
-            <origin xyz="0.0000267575 0.0000021499 0.0000258840" rpy="0 0 0"/>
-            <mass value="0.1700"/>
-            <inertia ixx="7.403494e-05"  ixy="5.337393e-06"  ixz="1.511932e-05"
-                                            iyy="1.426408e-04"  iyz="1.752534e-06"
-                                                                izz="1.672852e-04"/>
-        </inertial>
-        <visual>
-            <geometry>
-                <mesh filename="package://bumperbot_description/meshes/new_laser_link.stl"/>
-            </geometry>
-            <origin xyz="0 0 0" rpy="0 0 0"/>
-            <material name="dark_grey"/>
-        </visual>
-        <collision>
-            <geometry>
-                <box size="0.071689 0.097337 0.05350"/>
-            </geometry>
-            <origin xyz="0 0 -0.015" rpy="0 0 0"/>
-        </collision>
+      <inertial>
+        <origin xyz="0.0000267575 0.0000021499 0.0000258840" rpy="0 0 0"/>
+        <mass value="0.1700"/>
+        <inertia ixx="7.403494e-05"  ixy="5.337393e-06"  ixz="1.511932e-05"
+                                        iyy="1.426408e-04"  iyz="1.752534e-06"
+                                                            izz="1.672852e-04"/>
+      </inertial>
+      <visual>
+        <geometry>
+          <mesh filename="package://bumperbot_description/meshes/new_laser_link.stl"/>
+        </geometry>
+        <origin xyz="0 0 0" rpy="0 0 0"/>
+        <material name="dark_grey"/>
+      </visual>
+      <collision>
+        <geometry>
+          <box size="0.071689 0.097337 0.05350"/>
+        </geometry>
+        <origin xyz="0 0 -0.015" rpy="0 0 0"/>
+      </collision>
     </link>
   <joint name="laser_joint" type="fixed">
-        <origin xyz="0 0 0.131" rpy="0 0 0" /> <!-- z= 0.042(from physical unit) + 0.088(from fusion final assembly without wheels) + 0.001(accounting for plate thickness)-->
+        <origin xyz="0 0 0.131" rpy="0 0 3.14" /> <!-- z= 0.042(from physical unit) + 0.088(from fusion final assembly without wheels) + 0.001(accounting for plate thickness)-->
         <parent link="base_link" />
         <child link="laser" />

Commit message: laser is working added support for gz_bridge also.... found bug in link naming of laser... changed "laser" to "laser_link" everything is working, no bugs discovered

File: src/bumperbot_description/urdf/bumperbot.urdf.xacro (robot description, xacro)
@@ -147,5 +147,5 @@
     <child link="caster_rear_link" />
   </joint>
-  <link name="laser">
+  <link name="laser_link">
       <inertial>
         <origin xyz="0.0000267575 0.0000021499 0.0000258840" rpy="0 0 0"/>
@@ -172,5 +172,5 @@
         <origin xyz="0 0 0.131" rpy="0 0 3.14" /> <!-- z= 0.042(from physical unit) + 0.088(from fusion final assembly without wheels) + 0.001(accounting for plate thickness)-->
         <parent link="base_link" />
-        <child link="laser" />
+        <child link="laser_link" />
   </joint>
   <link name="imu_link">

File: src/bumperbot_description/urdf/bumperbot_gazebo.xacro (robot description, xacro)
@@ -44,5 +44,9 @@
         <parameters>$(find bumperbot_controller)/config/bumperbot_controllers.yaml</parameters>
       </plugin>
-      <plugin filename="ignition-gazebo-imu-system" name="ignition::gazebo::systems::Imu"></plugin>
+      <plugin filename="ignition-gazebo-imu-system" name="ignition::gazebo::systems::Imu">
+      </plugin>
+      <plugin filename="ignition-gazebo-sensors-system" name="ignition::gazebo::systems::Sensors">
+        <render_engine>ogre2</render_engine>
+      </plugin>
     </xacro:if>
     <!-- ROS 2 Iron or above -->
@@ -51,8 +55,12 @@
         <parameters>$(find bumperbot_controller)/config/bumperbot_controllers.yaml</parameters>
       </plugin>
-      <plugin filename="gz-sim-imu-system" name="gz::sim::systems::Imu"></plugin>
+      <plugin filename="gz-sim-imu-system" name="gz::sim::systems::Imu">
+      </plugin>
+      <plugin filename="gz-sim-sensors-system" name="gz::sim::systems::Sensors">
+        <render_engine>ogre2</render_engine>
+      </plugin>
     </xacro:unless>
   </gazebo>
-    <!-- IMU -->
+  <!-- IMU -->
   <gazebo reference="imu_link">
     <sensor name="imu" type="imu">
@@ -105,3 +113,33 @@
     </sensor>
   </gazebo>
+  <!-- 2D Laser Sensor -->
+  <gazebo reference="laser_link">
+    <sensor name="lidar" type="gpu_lidar">
+      <always_on>true</always_on>
+      <visualize>true</visualize>
+      <topic>scan</topic>
+      <update_rate>5</update_rate>
+      <gz_frame_id>laser_link</gz_frame_id>
+      <lidar>
+        <scan>
+          <horizontal>
+            <samples>360</samples>
+            <resolution>1.00000</resolution>
+            <min_angle>0.000000</min_angle>
+            <max_angle>6.280000</max_angle>
+          </horizontal>
+        </scan>
+        <range>
+          <min>0.120000</min>
+          <max>12.0</max>
+          <resolution>0.02</resolution>
+        </range>
+        <noise>
+          <type>gaussian</type>
+          <mean>0.0</mean>
+          <stddev>0.01</stddev>
+        </noise>
+      </lidar>
+    </sensor>
+  </gazebo>
 </robot>
