Commit message: fixed error,not tested using key_teleop

File: src/bumperbot_description/urdf/bumperbot.urdf.xacro (robot description, xacro)
@@ -59,5 +59,5 @@
   </link>
    <joint name="wheel_right_joint" type="continuous">
-    <origin xyz="0 0.16513032 0.035" rpy="0 0 0" />
+    <origin xyz="0 0.16513032 0.028" rpy="0 0 0" />
     <parent link="base_link" />
     <child link="wheel_right_link" />
@@ -88,5 +88,5 @@
   </link>
    <joint name="wheel_left_joint" type="continuous">
-    <origin xyz="0 -0.16513032 0.035" rpy="0 0 0" />
+    <origin xyz="0 -0.16513032 0.028" rpy="0 0 0" />
     <parent link="base_link" />
     <child link="wheel_left_link" />

Commit message: found small bug in imu placement, fixed

File: src/bumperbot_description/urdf/bumperbot.urdf.xacro (robot description, xacro)
@@ -197,5 +197,5 @@
     <parent link="base_link"/>
     <child link="imu_link"/>
-  <origin xyz="0.0 0.008 0.07" rpy="0.0 0.0 0.0"/> <!--x and y values from fusion and z value is from fusion but also adjusted -->
+  <origin xyz="0.0 0.008 0.071486" rpy="0.0 0.0 0.0"/> <!--x and y values from fusion and z value is from fusion but also adjusted -->
   </joint>
   <material name="blue">

Commit message: Update parameters and launch files to enable simulated time across various components, slam is working in simulation, yet to test in robot

File: src/bumperbot_description/urdf/bumperbot.urdf.xacro (robot description, xacro)
@@ -36,5 +36,5 @@
     <origin xyz="0 0 0.02434923" rpy="0 0 0"/>
   </joint>
-  <link name="wheel_right_link">
+  <link name="wheel_left_link">
    <inertial>
       <origin xyz="0 9.713661142e-10 0.016398450" rpy="0 0 0" />
@@ -48,5 +48,5 @@
       <material name="blue" />
       <geometry>
-        <mesh filename="package://bumperbot_description/meshes/wheel_right_link.stl"/>
+        <mesh filename="package://bumperbot_description/meshes/wheel_left_link.stl"/>
       </geometry>
     </visual>
@@ -58,12 +58,12 @@
     </collision>
   </link>
-   <joint name="wheel_right_joint" type="continuous">
+   <joint name="wheel_left_joint" type="continuous">
     <origin xyz="0 0.16513032 0.028" rpy="0 0 0" />
     <parent link="base_link" />
-    <child link="wheel_right_link" />
+    <child link="wheel_left_link" />
     <axis xyz="0 1 0" />
   </joint>
   <link
-    name="wheel_left_link">
+    name="wheel_right_link">
     <inertial>
       <origin xyz="0 9.713661142e-10 0.016398450" rpy="0 0 0" />
@@ -77,5 +77,5 @@
       <material name="blue" />
       <geometry>
-        <mesh filename="package://bumperbot_description/meshes/wheel_left_link.stl"/>
+        <mesh filename="package://bumperbot_description/meshes/wheel_right_link.stl"/>
       </geometry>
     </visual>
@@ -87,8 +87,8 @@
     </collision>
   </link>
-   <joint name="wheel_left_joint" type="continuous">
+   <joint name="wheel_right_joint" type="continuous">
     <origin xyz="0 -0.16513032 0.028" rpy="0 0 0" />
     <parent link="base_link" />
-    <child link="wheel_left_link" />
+    <child link="wheel_right_link" />
     <axis xyz="0 1 0" />
   </joint>

Commit message: changed urdf to match instrcutor's

File: src/bumperbot_description/urdf/bumperbot.urdf.xacro (robot description, xacro)
@@ -36,4 +36,33 @@
     <origin xyz="0 0 0.02434923" rpy="0 0 0"/>
   </joint>
+  <link
+    name="wheel_right_link">
+    <inertial>
+      <origin xyz="0 9.713661142e-10 0.016398450" rpy="0 0 0" />
+      <mass value="0.092049771" />
+      <inertia ixx="0.000093607"  ixy="0"  ixz="0"
+               iyy="0.000093607"  iyz="0"
+               izz="0.000180163" />
+    </inertial>
+    <visual>
+      <origin xyz="0 0 0" rpy="-1.57 0 0" />
+      <material name="blue" />
+      <geometry>
+        <mesh filename="package://bumperbot_description/meshes/wheel_right_link.stl"/>
+      </geometry>
+    </visual>
+    <collision>
+      <origin xyz="0 0.0146 0" rpy="-1.57 0 0" />
+      <geometry>
+        <cylinder radius="0.0534" length="0.0285"/>
+      </geometry>
+    </collision>
+  </link>
+   <joint name="wheel_right_joint" type="continuous">
+    <origin xyz="0 -0.16513032 0.028" rpy="0 0 0" />
+    <parent link="base_link" />
+    <child link="wheel_right_link" />
+    <axis xyz="0 1 0" />
+  </joint>
   <link name="wheel_left_link">
    <inertial>
@@ -62,33 +91,4 @@
     <parent link="base_link" />
     <child link="wheel_left_link" />
-    <axis xyz="0 1 0" />
-  </joint>
-  <link
-    name="wheel_right_link">
-    <inertial>
-      <origin xyz="0 9.713661142e-10 0.016398450" rpy="0 0 0" />
-      <mass value="0.092049771" />
-      <inertia ixx="0.000093607"  ixy="0"  ixz="0"
-               iyy="0.000093607"  iyz="0"
-               izz="0.000180163" />
-    </inertial>
-    <visual>
-      <origin xyz="0 0 0" rpy="-1.57 0 0" />
-      <material name="blue" />
-      <geometry>
-        <mesh filename="package://bumperbot_description/meshes/wheel_right_link.stl"/>
-      </geometry>
-    </visual>
-    <collision>
-      <origin xyz="0 0.0146 0" rpy="-1.57 0 0" />
-      <geometry>
-        <cylinder radius="0.0534" length="0.0285"/>
-      </geometry>
-    </collision>
-  </link>
-   <joint name="wheel_right_joint" type="continuous">
-    <origin xyz="0 -0.16513032 0.028" rpy="0 0 0" />
-    <parent link="base_link" />
-    <child link="wheel_right_link" />
     <axis xyz="0 1 0" />
   </joint>

Commit message: modified urdf for lidar to fit on downward side of robot, TODO: make new wheels and replace old wheels as lidar is touching ground

File: src/bumperbot_description/urdf/bumperbot.urdf.xacro (robot description, xacro)
@@ -170,5 +170,5 @@
   </link>
   <joint name="laser_joint" type="fixed">
-       <origin xyz="0 0 0.109" rpy="0 0 0" /> <!--z= 0.042(from physical unit) + 0.088(from fusion final assembly without wheels) + 0.001(accounting for plate thickness)-->
+        <origin xyz="0 0 0.0051" rpy="3.14159265 0 0" /> <!--z= 0.042(from physical unit) + 0.088(from fusion final assembly without wheels) + 0.001(accounting for plate thickness)-->
         <parent link="base_link" />
         <child link="laser_link" />

Commit message: Revert codebase state to match commit 7939855

File: src/bumperbot_description/urdf/bumperbot.urdf.xacro (robot description, xacro)
@@ -170,5 +170,5 @@
   </link>
   <joint name="laser_joint" type="fixed">
-        <origin xyz="0 0 0.0051" rpy="3.14159265 0 0" /> <!--z= 0.042(from physical unit) + 0.088(from fusion final assembly without wheels) + 0.001(accounting for plate thickness)-->
+       <origin xyz="0 0 0.109" rpy="0 0 0" /> <!--z= 0.042(from physical unit) + 0.088(from fusion final assembly without wheels) + 0.001(accounting for plate thickness)-->
         <parent link="base_link" />
         <child link="laser_link" />

File: src/bumperbot_description/urdf/test.urdf.xacro (robot description, xacro)
@@ -3,214 +3,190 @@
   <!-- Start GZ or Ignition depending on ROS 2 Version -->
   <xacro:arg name="is_ignition" default="true"/>
-  <xacro:arg name="is_sim" default="true"/>
   <!-- Include Gazebo Parameters -->
   <xacro:include filename="$(find bumperbot_description)/urdf/bumperbot_gazebo.xacro" />
   <!-- Include ros2_control Plugins -->
   <xacro:include filename="$(find bumperbot_description)/urdf/bumperbot_ros2_control.xacro" />
-  <link name="base_footprint"/>
+  <link name="base_footprint" />
   <link name="base_link">
     <inertial>
-      <origin xyz="-0.008675826 0.003144972 0.032628778" rpy="0 0 0"/>
-      <mass value="2.210665107"/>
-      <inertia ixx="0.011527704"    ixy="-5.335634932e-7"  ixz="-0.000228605"
-               iyy="0.005806872"    iyz="-0.000372021"
-               izz="0.014234404" />
+        <origin xyz="0.0065 0.002607 0.020274" rpy="0 0 0"/>
+        <mass value="0.947792"/>
+        <inertia ixx="3.036"    ixy="-0.4767"  ixz="-0.511"
+                 iyy="1.659"    iyz="-1.036"
+                 izz="3.374"/>
     </inertial>
     <visual>
-      <origin xyz="0 0 0.0015" rpy="0 0 0" />
-      <!-- <material name="black"/> -->
-      <geometry>
-        <mesh filename="package://bumperbot_description/meshes/base_link.stl"/>
-      </geometry>
+      <origin xyz="0 0 0.0015" rpy="0 0 1.57"/>
+        <geometry>
+            <mesh filename="package://bumperbot_description/meshes/base_link.stl" scale="0.001 0.001 0.001"/>
+        </geometry>
+        <material name="black"/>
     </visual>
     <collision>
-      <origin xyz="0 0 0.0015" rpy="0 0 0" />
-      <geometry>
-        <mesh filename="package://bumperbot_description/meshes/base_link.stl"/>
-      </geometry>
+        <origin xyz="0 0 0.0015" rpy="0 0 1.57"/>
+        <geometry>
+            <mesh filename="package://bumperbot_description/meshes/base_link.stl" scale="0.001 0.001 0.001"/>
+        </geometry>
     </collision>
   </link>
   <joint name="base_joint" type="fixed">
     <parent link="base_footprint"/>
-    <child link="base_link" />
-    <origin xyz="0 0 0.02434923" rpy="0 0 0"/>
+    <child link="base_link"/>
+    <origin xyz="0 0 0.038" rpy="0 0 0"/>
   </joint>
-  <link
-    name="wheel_right_link">
+  <link name="wheel_right_link">
     <inertial>
-      <origin xyz="0 9.713661142e-10 0.016398450" rpy="0 0 0" />
-      <mass value="0.092049771" />
-      <inertia ixx="0.000093607"  ixy="0"  ixz="0"
-               iyy="0.000093607"  iyz="0"
-               izz="0.000180163" />
-    </inertial>
-    <visual>
-      <origin xyz="0 0 0" rpy="-1.57 0 0" />
-      <material name="blue" />
-      <geometry>
-        <mesh filename="package://bumperbot_description/meshes/wheel_right_link.stl"/>
-      </geometry>
-    </visual>
-    <collision>
-      <origin xyz="0 0.0146 0" rpy="-1.57 0 0" />
-      <geometry>
-        <cylinder radius="0.0534" length="0.0285"/>
-      </geometry>
-    </collision>
-  </link>
-   <joint name="wheel_right_joint" type="continuous">
-    <origin xyz="0 -0.16513032 0.028" rpy="0 0 0" />
-    <parent link="base_link" />
-    <child link="wheel_right_link" />
-    <axis xyz="0 1 0" />
-  </joint>
-  <link name="wheel_left_link">
-   <inertial>
-      <origin xyz="0 9.713661142e-10 0.016398450" rpy="0 0 0" />
-      <mass value="0.092049771" />
-      <inertia ixx="0.000093607"  ixy="0"  ixz="0"
-               iyy="0.000093607"  iyz="0"
-               izz="0.000180163" />
-    </inertial>
-    <visual>
-      <origin xyz="0 0 0" rpy="1.57 0 0" />
-      <material name="blue" />
-      <geometry>
-        <mesh filename="package://bumperbot_description/meshes/wheel_left_link.stl"/>
-      </geometry>
-    </visual>
-    <collision>
-      <origin xyz="0 -0.0146 0" rpy="1.57 0 0" />
-      <geometry>
-        <cylinder radius="0.0534" length="0.0285"/>
-      </geometry>
-    </collision>
-  </link>
-   <joint name="wheel_left_joint" type="continuous">
-    <origin xyz="0 0.16513032 0.028" rpy="0 0 0" />
-    <parent link="base_link" />
-    <child link="wheel_left_link" />
-    <axis xyz="0 1 0" />
-  </joint>
-  <link name="caster_front_link">
-    <inertial>
-      <origin xyz="5.375138993e-07 -9.84538264e-07 0.012447006" rpy="0 0 0" />
-      <mass value="0.006654822" />
-      <inertia ixx="5.314741443e-07"  ixy="0.00"    ixz="0.00"
-               iyy="4.867361117e-07"  iyz="0.00"
-               izz="4.568100217e-07" />
-    </inertial>
-    <visual>
-      <origin xyz="0 0 0" rpy="0 0 1.57" />
-      <material name="silver"/>
-      <geometry>
-        <mesh filename="package://bumperbot_description/meshes/caster_front_link.stl"/>
-      </geometry>
-    </visual>
-    <collision>
-      <origin xyz="0 0 0.01240923" rpy="0 0 1.57" />
-      <geometry>
-        <sphere radius="0.013004615"/>
-      </geometry>
-    </collision>
-  </link>
-  <joint name="caster_front_joint" type="fixed">
-    <origin xyz="0.1101000 0.00074129 -0.02450923" rpy="0 0 0" />
-    <parent link="base_link" />
-    <child link="caster_front_link" />
-  </joint>
-  <link name="caster_rear_link">
-    <inertial>
-      <origin xyz="5.375138993e-07 -9.84538264e-07 0.012447006" rpy="0 0 0" />
-      <mass value="0.006654822" />
-      <inertia ixx="5.314741443e-07"  ixy="0.00"    ixz="0.00"
-               iyy="4.867361117e-07"  iyz="0.00"
-               izz="4.568100217e-07" />
-    </inertial>
-    <visual>
-      <origin xyz="0 0 0" rpy="0 0 1.57" />
-      <material name="silver"/>
-      <geometry>
-        <mesh filename="package://bumperbot_description/meshes/caster_rear_link.stl"/>
-      </geometry>
-    </visual>
-    <collision>
-      <origin xyz="0 0 0.01240923" rpy="0 0 1.57" />
-      <geometry>
-        <sphere radius="0.013004615"/>
-      </geometry>
-    </collision>
-  </link>
-  <joint name="caster_rear_joint" type="fixed">
-    <origin xyz="-0.1101000 0.00074129 -0.02450923" rpy="0 0 0" />
-    <parent link="base_link" />
-    <child link="caster_rear_link" />
-  </joint>
-  <link name="laser_link">
-      <inertial>
-        <origin xyz="0.0000267575 0.0000021499 0.0000258840" rpy="0 0 0"/>
-        <mass value="0.1700"/>
-        <inertia ixx="7.403494e-05"  ixy="5.337393e-06"  ixz="1.511932e-05"
-                                     iyy="1.426408e-04"  iyz="1.752534e-06"
-                                                            izz="1.672852e-04"/>
-      </inertial>
-      <visual>
-        <geometry>
-          <mesh filename="package://bumperbot_description/meshes/laser_link.stl"/>
-        </geometry>
-        <origin xyz="0 0 0" rpy="0 0 3.14"/>
-        <material name="dark_grey"/>
-      </visual>
-      <collision>
-        <origin xyz="0 0 0.03150" rpy="0 0 3.14"/>
-        <geometry>
-          <box size="0.071689 0.097337 0.05350"/>
-        </geometry>
-      </collision>
-  </link>
-  <joint name="laser_joint" type="fixed">
-       <origin xyz="0 0 0.109" rpy="0 0 0" /> <!--z= 0.042(from physical unit) + 0.088(from fusion final assembly without wheels) + 0.001(accounting for plate thickness)-->
+        <origin xyz="6.671e-12 -1.094e-11 0.012102" rpy="0 0 0"/>
+        <mass value="0.09205"/>
+        <inertia ixx="9.3607e-05"  ixy="-4.428e-15"  ixz="6.941e-16"
+                                    iyy="9.3607e-05"  iyz="-1.133e-15"
+                                                        izz="1.802e-04"/>
+        </inertial>
+        <visual>
+            <geometry>
+                <mesh filename="package://bumperbot_description/meshes/c.stl" scale="0.001 0.001 0.001"/>
+            </geometry>
+            <origin xyz="0 0 0" rpy="-1.57 0 0"/>
+            <material name="blue" />
+        </visual>
+        <collision>
+            <geometry>
+                <mesh filename="package://bumperbot_description/meshes/wheel_right_link.stl" scale="0.001 0.001 0.001"/>
+            </geometry>
+            <origin xyz="0 0 0" rpy="-1.57 0 0"/>
+            <material name="blue" />
+        </collision>
+    </link>
+    <joint name="wheel_right_joint" type="continuous">
+        <origin xyz="0 -0.14355 0.015" rpy="0 0 0" />
         <parent link="base_link" />
-        <child link="laser_link" />
-  </joint>
-  <link name="imu_link">
-    <inertial>
-      <origin xyz="-0.057000001 -0.076500001 0.048500000" rpy="0.0 0.0 0.0"/>
-      <mass value="0.001307313"/>
-      <inertia ixx="4.630065354e-08" ixy="0.0" ixz="0.0" iyy="2.723567855e-08" iyz="0.0" izz="6.808919639e-08"/>
-    </inertial>
-    <visual>
-      <origin xyz="0 0 0" rpy="0 0 0" />
-      <material name="amber_gold"/>
-      <geometry>
-        <mesh filename="package://bumperbot_description/meshes/imu_link_new.stl"/>
-      </geometry>
-    </visual>
-    <collision>
-      <origin xyz="0 0 0" rpy="0 0 0" />
-      <geometry>
-        <box size="0.02 0.015 0.005"/>
-      </geometry>
-    </collision>
-  </link>
-  <joint name="imu_joint" type="fixed">
-    <parent link="base_link"/>
-    <child link="imu_link"/>
-  <origin xyz="0.0 0.008 0.071486" rpy="0.0 0.0 0.0"/> <!--x and y values from fusion and z value is from fusion but also adjusted -->
-  </joint>
-  <material name="blue">
-    <color rgba="0 0 1 1"/>
-  </material>
-  <material name="black">
-    <color rgba="0 0 0 1"/>
-  </material>
-  <material name="silver">
-    <color rgba="0.79 0.82 0.93 1"/>
-  </material>
-  <material name="dark_grey">
-    <color rgba="0.3 0.3 0.3 1"/>
-  </material>
-  <material name="amber_gold">
-    <color rgba="1.0 0.75 0.0 1.0"/>
-  </material>
+        <child link="wheel_right_link" />
+        <axis xyz="0 1 0" />
+    </joint>
+    <link name="wheel_left_link">
+        <inertial>
+        <origin xyz="6.671e-12 -1.094e-11 0.012102" rpy="0 0 0"/>
+        <mass value="0.09205"/>
+        <inertia ixx="9.3607e-05"  ixy="-4.428e-15"  ixz="6.941e-16"
+                                    iyy="9.3607e-05"  iyz="-1.133e-15"
+                                                        izz="1.802e-04"/>
+        </inertial>
+        <visual>
+            <geometry>
+                <mesh filename="package://bumperbot_description/meshes/wheel_left_link.stl" scale="0.001 0.001 0.001"/>
+            </geometry>
+            <origin xyz="0 0 0" rpy="1.57 0 0"/>
+            <material name="blue" />
+        </visual>
+        <collision>
+            <geometry>
+                <mesh filename="package://bumperbot_description/meshes/wheel_left_link.stl" scale="0.001 0.001 0.001"/>
+            </geometry>
+            <origin xyz="0 0 0" rpy="1.57 0 0"/>
+            <material name="blue" />
+        </collision>
+    </link>
+    <joint name="wheel_left_joint" type="continuous">
+        <origin xyz="0 0.14355 0.015" rpy="0 0 0" /> <!-- z value = height of protruded part of wheel(long) from fusion assembly-->
+        <!-- y value = (-0.12855 - 0.015) where 0.015 is height of protruded part of wheel(long) from fusion assembly and the 0.12855 is radius of base plate + approximation of around 0.5inches-->
+        <parent link="base_link" />
+        <child link="wheel_left_link" />
+        <axis xyz="0 1 0" />
+    </joint>
+    <link name="caster_front_link">
+        <inertial>
+        <origin xyz="0.000348 -0.003895 0.018625" rpy="0 0 0"/>
+        <mass value="0.030003"/>
+        <inertia ixx="5.032352e-06"  ixy="7.6e-10"    ixz="-5.91e-10"
+                                        iyy="5.178243e-06"  iyz="-2.92e-10"
+                                                            izz="5.249228e-06"/>
+        </inertial>
+        <visual>
+            <geometry>
+                <mesh filename="package://bumperbot_description/meshes/caster_front_link.stl" scale="0.001 0.001  0.001"/>
+            </geometry>
+            <origin xyz="0 0 0" rpy="0 0 1.57"/>
+            <material name="silver"/>
+        </visual>
+        <collision>
+            <geometry>
+                <mesh filename="package://bumperbot_description/meshes/caster_front_link.stl" scale="0.001 0.001  0.001"/>
+            </geometry>
+            <origin xyz="0 0 0" rpy="0 0 1.57"/>
+        </collision>
+    </link>
+    <joint name="caster_front_joint" type="fixed">
+        <origin xyz="0.0762 0 -0.0395011" rpy="0 0 0" /> <!-- x value = 3 inches   y value = from fusion caster height-->
+        <parent link="base_link" />
+        <child link="caster_front_link" />
+    </joint>
+    <link name="caster_rear_link">
+        <inertial>
+        <origin xyz="0.000348 -0.003895 0.018625" rpy="0 0 0"/>
+        <mass value="0.030003"/>
+        <inertia ixx="5.032352e-06"  ixy="7.6e-10"    ixz="-5.91e-10"
+                                        iyy="5.178243e-06"  iyz="-2.92e-10"
+                                                            izz="5.249228e-06"/>
+        </inertial>
+        <visual>
+            <geometry>
+                <mesh filename="package://bumperbot_description/meshes/caster_rear_link.stl" scale="0.001 0.001  0.001"/>
+            </geometry>
+            <origin xyz="0 0 0" rpy="0 0 1.57"/>
+            <material name="silver"/>
+        </visual>
+        <collision>
+            <geometry>
+                <mesh filename="package://bumperbot_description/meshes/caster_rear_link.stl" scale="0.001 0.001  0.001"/>
+            </geometry>
+            <origin xyz="0 0 0" rpy="0 0 1.57"/>
+        </collision>
+    </link>
+    <joint name="caster_rear_joint" type="fixed">
+        <origin xyz="-0.0762 0 -0.0395011" rpy="0 0 0" /> <!-- x value = 3 inches   y value = from fusion caster height-->
+        <parent link="base_link" />
+        <child link="caster_rear_link" />
+    </joint>
+    <link name="laser">
+        <inertial>
+            <origin xyz="0.0000267575 0.0000021499 0.0000258840" rpy="0 0 0"/>
+            <mass value="0.1700"/>
+            <inertia ixx="7.403494e-05"  ixy="5.337393e-06"  ixz="1.511932e-05"
+                                            iyy="1.426408e-04"  iyz="1.752534e-06"
+                                                                izz="1.672852e-04"/>
+        </inertial>
+        <visual>
+            <geometry>
+                <mesh filename="package://bumperbot_description/meshes/new_laser_link.stl"/>
+            </geometry>
+            <origin xyz="0 0 0" rpy="0 0 0"/>
+            <material name="dark_grey"/>
+        </visual>
+        <collision>
+            <geometry>
+                <mesh filename="package://bumperbot_description/meshes/new_laser_link.stl"/>
+            </geometry>
+            <origin xyz="0 0 0" rpy="0 0 0"/>
+        </collision>
+    </link>
+    <joint name="laser_joint" type="fixed">
+        <origin xyz="0 0 0.131" rpy="0 0 0" /> <!-- z= 0.042(from physical unit) + 0.088(from fusion final assembly without wheels) + 0.001(accounting for plate thickness)-->
+        <parent link="base_link" />
+        <child link="laser" />
+    </joint>
+    <material name="blue">
+        <color rgba="0 0 1 1"/>
+    </material>
+    <material name="black">
+        <color rgba="0 0 0 1"/>
+    </material>
+    <material name="silver">
+        <color rgba="0.79 0.82 0.93 1"/>
+    </material>
+    <material name="dark_grey">
+        <color rgba="0.3 0.3 0.3 1"/>
+    </material>
+    <material name="amber_gold">
+        <color rgba="1.0 0.75 0.0 1.0"/>
+    </material>
 </robot>
